Commit message: feat: Replace old bdx_r robot model with new version
This commit replaces the entire old robot URDF and assets with the new version.

File: robots/bdx_r/bdx_r.urdf (robot description, URDF)
Before this commit: robot rob_bdx, 20 links, 19 joints
Links:
- removed link battery_2
- removed link left_foot_pad_1
- removed link left_hip_1
- removed link left_hip_connector_1
- removed link left_hip_rotator_1
- removed link left_lower_leg_1
- removed link left_upper_leg_1
- removed link neck_motor_1
- removed link right_foot_pad_1
- removed link right_hip_1
- removed link right_hip_connector_2
- removed link right_hip_rotator_1
- removed link right_lower_leg_2
- removed link right_upper_leg_2
- added link Antenna, mass 0.02; collision mesh filename=assets/Antenna.stl scale=0.001 0.001 0.001; visual mesh filename=assets/Antenna.stl scale=0.001 0.001 0.001
- added link AntennaBox, mass 0.065; collision mesh filename=assets/AntennaBox.stl scale=0.001 0.001 0.001; visual mesh filename=assets/AntennaBox.stl scale=0.001 0.001 0.001
- added link BackCover, mass 0.35; collision mesh filename=assets/BackCover.stl scale=0.001 0.001 0.001; visual mesh filename=assets/BackCover.stl scale=0.001 0.001 0.001
- added link BackFrame, mass 0.1; collision mesh filename=assets/BackFrame.stl scale=0.001 0.001 0.001; visual mesh filename=assets/BackFrame.stl scale=0.001 0.001 0.001
- added link Battery, mass 1.00; collision mesh filename=assets/Battery.stl scale=0.001 0.001 0.001; visual mesh filename=assets/Battery.stl scale=0.001 0.001 0.001
- added link BottomCover, mass 0.03; collision mesh filename=assets/BottomCover.stl scale=0.001 0.001 0.001; visual mesh filename=assets/BottomCover.stl scale=0.001 0.001 0.001
- added link FrontCover, mass 0.4; collision mesh filename=assets/FrontCover.stl scale=0.001 0.001 0.001; visual mesh filename=assets/FrontCover.stl scale=0.001 0.001 0.001
- added link IMU_Mount, mass 0.02; collision mesh filename=assets/IMU_Mount.stl scale=0.001 0.001 0.001; visual mesh filename=assets/IMU_Mount.stl scale=0.001 0.001 0.001
- added link Jetson_Mount, mass 0.3; collision mesh filename=assets/Jetson_Mount.stl scale=0.001 0.001 0.001; visual mesh filename=assets/Jetson_Mount.stl scale=0.001 0.001 0.001
- added link LeftAnkleCover, mass 0.01; collision mesh filename=assets/LeftAnkleCover.stl scale=0.001 0.001 0.001; visual mesh filename=assets/LeftAnkleCover.stl scale=0.001 0.001 0.001
- added link LeftBottomLegCover, mass 0.1; collision mesh filename=assets/LeftBottomLegCover.stl scale=0.001 0.001 0.001; visual mesh filename=assets/LeftBottomLegCover.stl scale=0.001 0.001 0.001
- added link LeftFootCover, mass 0.01; collision mesh filename=assets/LeftFootCover.stl scale=0.001 0.001 0.001; visual mesh filename=assets/LeftFootCover.stl scale=0.001 0.001 0.001
- added link LeftFootPad, mass 0.05; collision mesh filename=assets/LeftFootPad.stl scale=0.001 0.001 0.001; visual mesh filename=assets/LeftFootPad.stl scale=0.001 0.001 0.001
- added link LeftLegBottomPlug, mass 0.01; collision mesh filename=assets/LeftLegBottomPlug.stl scale=0.001 0.001 0.001; visual mesh filename=assets/LeftLegBottomPlug.stl scale=0.001 0.001 0.001
- added link LeftLegUpperPlug, mass 0.01; collision mesh filename=assets/LeftLegUpperPlug.stl scale=0.001 0.001 0.001; visual mesh filename=assets/LeftLegUpperPlug.stl scale=0.001 0.001 0.001
- added link LeftUpperLegCover, mass 0.1; collision mesh filename=assets/LeftUpperLegCover.stl scale=0.001 0.001 0.001; visual mesh filename=assets/LeftUpperLegCover.stl scale=0.001 0.001 0.001
- added link Left_Ankle_Motor, mass 0.3657589373000338; collision mesh filename=assets/Left_Ankle_Motor.stl scale=0.001 0.001 0.001; visual mesh filename=assets/Left_Ankle_Motor.stl scale=0.001 0.001 0.001
- added link Left_Hip_Connector, mass 0.15534729534246716; collision mesh filename=assets/Left_Hip_Connector.stl scale=0.001 0.001 0.001; visual mesh filename=assets/Left_Hip_Connector.stl scale=0.001 0.001 0.001
- added link Left_Hip_Pitch_Motor, mass 0.9104515144014014; collision mesh filename=assets/Left_Hip_Pitch_Motor.stl scale=0.001 0.001 0.001; visual mesh filename=assets/Left_Hip_Pitch_Motor.stl scale=0.001 0.001 0.001
- added link Left_Hip_Roll_Motor, mass 1.071352674987853; collision mesh filename=assets/Left_Hip_Roll_Motor.stl scale=0.001 0.001 0.001; visual mesh filename=assets/Left_Hip_Roll_Motor.stl scale=0.001 0.001 0.001
- added link Left_Hip_Yaw_Motor, mass 0.9104522842757782; collision mesh filename=assets/Left_Hip_Yaw_Motor.stl scale=0.001 0.001 0.001; visual mesh filename=assets/Left_Hip_Yaw_Motor.stl scale=0.001 0.001 0.001
- added link Left_Knee_Motor, mass 0.9104515169769222; collision mesh filename=assets/Left_Knee_Motor.stl scale=0.001 0.001 0.001; visual mesh filename=assets/Left_Knee_Motor.stl scale=0.001 0.001 0.001
- added link Left_Lower_Leg, mass 0.4; collision mesh filename=assets/Left_Lower_Leg.stl scale=0.001 0.001 0.001; visual mesh filename=assets/Left_Lower_Leg.stl scale=0.001 0.001 0.001
- added link Left_Upper_Leg, mass 0.5042346129898978; collision mesh filename=assets/Left_Upper_Leg.stl scale=0.001 0.001 0.001; visual mesh filename=assets/Left_Upper_Leg.stl scale=0.001 0.001 0.001
- added link Neck_Motor, mass 0.9104522776624081; collision mesh filename=assets/Neck_Motor.stl scale=0.001 0.001 0.001; visual mesh filename=assets/Neck_Motor.stl scale=0.001 0.001 0.001
- added link RightAnkleCover, mass 0.02; collision mesh filename=assets/RightAnkleCover.stl scale=0.001 0.001 0.001; visual mesh filename=assets/RightAnkleCover.stl scale=0.001 0.001 0.001
- added link RightBottomLegCover, mass 0.1; collision mesh filename=assets/RightBottomLegCover.stl scale=0.001 0.001 0.001; visual mesh filename=assets/RightBottomLegCover.stl scale=0.001 0.001 0.001
- added link RightFootCover, mass 0.02; collision mesh filename=assets/RightFootCover.stl scale=0.001 0.001 0.001; visual mesh filename=assets/RightFootCover.stl scale=0.001 0.001 0.001
- added link RightFootPad, mass 0.05; collision mesh filename=assets/RightFootPad.stl scale=0.001 0.001 0.001; visual mesh filename=assets/RightFootPad.stl scale=0.001 0.001 0.001
- added link RightLegBottomPlug, mass 0.01; collision mesh filename=assets/RightLegBottomPlug.stl scale=0.001 0.001 0.001; visual mesh filename=assets/RightLegBottomPlug.stl scale=0.001 0.001 0.001
- added link RightLegUpperPlug, mass 0.01; collision mesh filename=assets/RightLegUpperPlug.stl scale=0.001 0.001 0.001; visual mesh filename=assets/RightLegUpperPlug.stl scale=0.001 0.001 0.001
- added link RightUpperLegCover, mass 0.1; collision mesh filename=assets/RightUpperLegCover.stl scale=0.001 0.001 0.001; visual mesh filename=assets/RightUpperLegCover.stl scale=0.001 0.001 0.001
- added link Right_Ankle_Motor, mass 0.3657591169602799; collision mesh filename=assets/Right_Ankle_Motor.stl scale=0.001 0.001 0.001; visual mesh filename=assets/Right_Ankle_Motor.stl scale=0.001 0.001 0.001
- added link Right_Hip_Connector, mass 0.15534729534247135; collision mesh filename=assets/Right_Hip_Connector.stl scale=0.001 0.001 0.001; visual mesh filename=assets/Right_Hip_Connector.stl scale=0.001 0.001 0.001
- added link Right_Hip_Pitch_Motor, mass 0.9104522697583138; collision mesh filename=assets/Right_Hip_Pitch_Motor.stl scale=0.001 0.001 0.001; visual mesh filename=assets/Right_Hip_Pitch_Motor.stl scale=0.001 0.001 0.001
- added link Right_Hip_Roll_Motor, mass 1.0713531089572514; collision mesh filename=assets/Right_Hip_Roll_Motor.stl scale=0.001 0.001 0.001; visual mesh filename=assets/Right_Hip_Roll_Motor.stl scale=0.001 0.001 0.001
- added link Right_Hip_Yaw_Motor, mass 0.9104522697579285; collision mesh filename=assets/Right_Hip_Yaw_Motor.stl scale=0.001 0.001 0.001; visual mesh filename=assets/Right_Hip_Yaw_Motor.stl scale=0.001 0.001 0.001
- added link Right_Knee_Motor, mass 0.9104522723338422; collision mesh filename=assets/Right_Knee_Motor.stl scale=0.001 0.001 0.001; visual mesh filename=assets/Right_Knee_Motor.stl scale=0.001 0.001 0.001
- added link Right_Lower_Leg, mass 0.4; collision mesh filename=assets/Right_Lower_Leg.stl scale=0.001 0.001 0.001; visual mesh filename=assets/Right_Lower_Leg.stl scale=0.001 0.001 0.001
- added link Right_Upper_Leg, mass 0.5042346187696303; collision mesh filename=assets/Right_Upper_Leg.stl scale=0.001 0.001 0.001; visual mesh filename=assets/Right_Upper_Leg.stl scale=0.001 0.001 0.001
- added link TopLeftCover, mass 0.1; collision mesh filename=assets/TopLeftCover.stl scale=0.001 0.001 0.001; visual mesh filename=assets/TopLeftCover.stl scale=0.001 0.001 0.001
- added link TopRightCover, mass 0.1; collision mesh filename=assets/TopRightCover.stl scale=0.001 0.001 0.001; visual mesh filename=assets/TopRightCover.stl scale=0.001 0.001 0.001
- link body_r: mass 13.680857694433165 -> 1.6; geometry collision mesh filename=assets/base_link.stl scale=0.001 0.001 0.001; visual mesh filename=assets/base_link.stl scale=0.001 0.001 0.001
- link left_foot_1: mass 1.6684693786230702 -> 0.22236469248575175; geometry collision mesh filename=assets/Left_Foot.stl scale=0.001 0.001 0.001; visual mesh filename=assets/Left_Foot.stl scale=0.001 0.001 0.001
- link right_foot_2: mass 1.668469378566157 -> 0.2223646924781009; geometry collision mesh filename=assets/Right_Foot.stl scale=0.001 0.001 0.001; visual mesh filename=assets/Right_Foot.stl scale=0.001 0.001 0.001
Joints:
- removed joint left_foot_pad
- removed joint right_foot_pad
- added joint Rigid 10: type fixed, parent body_r, child Jetson_Mount, origin xyz=0.076306 0.077202 0.016701 rpy=0 0 0
- added joint Rigid 11: type fixed, parent body_r, child Neck_Motor, origin xyz=0.076005 0.108952 0.134165 rpy=0 0 0
- added joint Rigid 12: type fixed, parent body_r, child Battery, origin xyz=0.0 -0.002881 0.093743 rpy=0 0 0
- added joint Rigid 13: type fixed, parent BackCover, child Antenna, origin xyz=-0.019105 0.0 -6e-06 rpy=0 0 0
- added joint Rigid 14: type fixed, parent Antenna, child AntennaBox, origin xyz=-0.008 0.0 0.0 rpy=0 0 0
- added joint Rigid 19: type fixed, parent Right_Hip_Pitch_Motor, child Right_Upper_Leg, origin xyz=0.018686 -0.0025 0.045297 rpy=0 0 0
- added joint Rigid 21: type fixed, parent Right_Upper_Leg, child Right_Knee_Motor, origin xyz=-0.052447 0.0 -0.104765 rpy=0 0 0
- added joint Rigid 23: type fixed, parent Right_Lower_Leg, child Right_Ankle_Motor, origin xyz=0.021506 0.00934 -0.102367 rpy=0 0 0
- added joint Rigid 24: type fixed, parent Right_Lower_Leg, child RightAnkleCover, origin xyz=0.07256 0.045378 -0.097474 rpy=0 0 0
- added joint Rigid 27: type fixed, parent right_foot_2, child RightFootCover, origin xyz=-0.041649 -0.0105 -0.042645 rpy=0 0 0
- added joint Rigid 28: type fixed, parent Right_Upper_Leg, child RightBottomLegCover, origin xyz=-0.14358 -0.0465 -0.112149 rpy=0 0 0
- added joint Rigid 29: type fixed, parent Right_Upper_Leg, child RightUpperLegCover, origin xyz=-0.008513 -0.0465 0.000589 rpy=0 0 0
- added joint Rigid 30: type fixed, parent RightUpperLegCover, child RightLegUpperPlug, origin xyz=-0.006969 -0.02025 -0.047727 rpy=0 0 0
- added joint Rigid 31: type fixed, parent RightBottomLegCover, child RightLegBottomPlug, origin xyz=0.06601 -0.02025 -0.009329 rpy=0 0 0
- added joint Rigid 33: type fixed, parent Left_Hip_Pitch_Motor, child Left_Upper_Leg, origin xyz=-0.018816 0.0025 0.045243 rpy=0 0 0
- added joint Rigid 34: type fixed, parent Left_Upper_Leg, child Left_Knee_Motor, origin xyz=-0.041231 0.0392 -0.077962 rpy=0 0 0
- added joint Rigid 36: type fixed, parent Left_Lower_Leg, child Left_Ankle_Motor, origin xyz=0.044852 -0.00934 -0.093516 rpy=0 0 0
- added joint Rigid 39: type fixed, parent left_foot_1, child LeftFootCover, origin xyz=-0.041648 0.0105 -0.042644 rpy=0 0 0
- added joint Rigid 40: type fixed, parent Left_Lower_Leg, child LeftAnkleCover, origin xyz=0.018114 -0.045377 -0.162552 rpy=0 0 0
- added joint Rigid 41: type fixed, parent Left_Upper_Leg, child LeftBottomLegCover, origin xyz=-0.106078 0.0465 -0.112095 rpy=0 0 0
- added joint Rigid 42: type fixed, parent Left_Upper_Leg, child LeftUpperLegCover, origin xyz=0.028989 0.0465 0.000643 rpy=0 0 0
- added joint Rigid 43: type fixed, parent LeftBottomLegCover, child LeftLegBottomPlug, origin xyz=0.06601 0.02025 -0.009329 rpy=0 0 0
- added joint Rigid 44: type fixed, parent LeftUpperLegCover, child LeftLegUpperPlug, origin xyz=-0.013452 0.02025 -0.033648 rpy=0 0 0
- added joint Rigid 5: type fixed, parent BackFrame, child BackCover, origin xyz=-0.066834 6.8e-05 -0.029977 rpy=0 0 0
- added joint Rigid 6: type fixed, parent body_r, child FrontCover, origin xyz=0.071231 -0.015041 0.058018 rpy=0 0 0
- added joint Rigid 7: type fixed, parent body_r, child TopLeftCover, origin xyz=-0.068283 0.178249 0.108311 rpy=0 0 0
- added joint Rigid 8: type fixed, parent body_r, child TopRightCover, origin xyz=-0.068283 -0.003845 0.108311 rpy=0 0 0
- added joint Rigid 9: type fixed, parent body_r, child IMU_Mount, origin xyz=-0.047178 0.066302 0.110944 rpy=0 0 0
- added joint left_foot_to_pad: type fixed, parent left_foot_1, child LeftFootPad, origin xyz=0.026824 -0.018025 -0.059089 rpy=0 0 0
- added joint right_foot_to_pad: type fixed, parent right_foot_2, child RightFootPad, origin xyz=0.026823 0.018026 -0.059089 rpy=0 0 0
- joint Rigid 1: child battery_2 -> Right_Hip_Yaw_Motor; origin xyz=0.0 -0.178361 0.018723 rpy=0 0 0 -> xyz=0.019472 0.018451 0.046444 rpy=0 0 0
- joint Rigid 2: child right_hip_rotator_1 -> Left_Hip_Yaw_Motor; origin xyz=0.05 -0.113 0.095944 rpy=0 0 0 -> xyz=0.019472 0.155954 0.046444 rpy=0 0 0
- joint Rigid 3: child left_hip_rotator_1 -> BottomCover; origin xyz=-0.05 -0.113 0.095944 rpy=0 0 0 -> xyz=0.002222 0.024202 -0.1018 rpy=0 0 0
- joint Rigid 4: child neck_motor_1 -> BackFrame; origin xyz=-0.023465 0.02175 0.086726 rpy=0 0 0 -> xyz=-0.096859 0.137077 0.060614 rpy=0 0 0
- joint left_ankle: axis -0.0 1.0 -0.0 -> -0.0 -1.0 -0.0; limit lower=-0.7 upper=1.26 effort=17 velocity=30 -> lower=-0.85 upper=1.3 effort=11.9 velocity=37.699; origin xyz=0.045148 -0.00584 -0.130078 rpy=0 0 0 -> xyz=0.00052 0.004 -0.036497 rpy=0 0 0; parent left_lower_leg_1 -> Left_Ankle_Motor
- joint left_foot_frame: parent left_foot_pad_1 -> LeftFootPad
- joint left_hip_pitch: axis 0.0 -1.0 0.0 -> -0.0 -1.0 0.0; child left_upper_leg_1 -> Left_Hip_Pitch_Motor; limit lower=-2.6 upper=1.9 effort=60 velocity=30 -> lower=-0.5 upper=1 effort=42 velocity=18.849; origin xyz=-0.03875 -0.166147 0.001341 rpy=0 0 0 -> xyz=-0.008647 0.07125 0.001341 rpy=0 0 0; parent left_hip_connector_1 -> Left_Hip_Connector
- joint left_hip_roll: axis -1.0 -0.0 0.0 -> 1.0 -0.0 0.0; child left_hip_connector_1 -> Left_Hip_Connector; limit lower=-0.3 upper=1.0 effort=60 velocity=30 -> lower=-0.3 upper=0.3 effort=42 velocity=18.849; parent left_hip_1 -> Left_Hip_Roll_Motor
- joint left_hip_yaw: axis 0.0 -0.0 1.0 -> 0.0 0.0 1.0; child left_hip_1 -> Left_Hip_Roll_Motor; limit lower=-0.4 upper=0.25 effort=60 velocity=30 -> lower=-0.5 upper=0.35 effort=42 velocity=18.849; origin xyz=-0.063 0.163 -0.052 rpy=0 0 0 -> xyz=-0.04527 -0.018752 -0.0025 rpy=0 0 0; parent left_hip_rotator_1 -> Left_Hip_Yaw_Motor
- joint left_knee: axis -0.0 1.0 -0.0 -> -0.0 -1.0 0.0; child left_lower_leg_1 -> Left_Lower_Leg; limit lower=-0.9 upper=1.2 effort=60 velocity=30 -> lower=-0.95 upper=1.2 effort=42.0 velocity=18.849; origin xyz=-0.049202 0.237397 -0.077709 rpy=0 0 0 -> xyz=-0.019146 -0.042 -0.045104 rpy=0 0 0; parent left_upper_leg_1 -> Left_Knee_Motor
- joint right_ankle: axis -0.0 1.0 0.0 -> 0.0 -1.0 0.0; limit lower=-0.7 upper=1.26 effort=60 velocity=30 -> lower=-1.3 upper=0.85 effort=11.9 velocity=37.699; origin xyz=0.04647 0.00584 -0.129612 rpy=0 0 0 -> xyz=0.023858 -0.004 -0.027623 rpy=0 0 0; parent right_lower_leg_2 -> Right_Ankle_Motor
- joint right_foot_frame: parent right_foot_pad_1 -> RightFootPad
- joint right_hip_pitch: axis 0.0 -1.0 -0.0 -> -0.0 -1.0 -0.0; child right_upper_leg_2 -> Right_Hip_Pitch_Motor; limit lower=-2.6 upper=1.9 effort=60 velocity=30 -> lower=-1 upper=0.5 effort=42 velocity=18.849; parent right_hip_connector_2 -> Right_Hip_Connector
- joint right_hip_roll: axis 1.0 0.0 0.0 -> -1.0 0.0 -0.0; child right_hip_connector_2 -> Right_Hip_Connector; limit lower=-0.3 upper=1.0 effort=60 velocity=30 -> lower=-0.3 upper=0.3 effort=42 velocity=18.849; parent right_hip_1 -> Right_Hip_Roll_Motor
- joint right_hip_yaw: axis 0.0 -0.0 -1.0 -> 0.0 0.0 1.0; child right_hip_1 -> Right_Hip_Roll_Motor; limit lower=-0.4 upper=0.25 effort=60 velocity=30 -> lower=-0.5 upper=0.35 effort=42 velocity=18.849; origin xyz=-0.163 0.063 -0.052 rpy=0 0 0 -> xyz=-0.04527 0.018751 -0.0025 rpy=0 0 0; parent right_hip_rotator_1 -> Right_Hip_Yaw_Motor
- joint right_knee: axis -0.0 1.0 0.0 -> -0.0 -1.0 -0.0; child right_lower_leg_2 -> Right_Lower_Leg; limit lower=-0.9 upper=1.2 effort=60 velocity=30 -> lower=-1.2 upper=0.95 effort=42 velocity=18.849; origin xyz=-0.078511 0.0 -0.078512 rpy=0 0 0 -> xyz=-0.045432 0.0025 -0.018355 rpy=0 0 0; parent right_upper_leg_2 -> Right_Knee_Motor
